File: board/BiasCircuit.kicad_sch (KiCad schematic)
At the start: 35 parts, among them U2 LTC4302-1, U3 AD5144_100k, U4 LT3080xDD, U5 AQY212G3HS, U6 INA219AxD

Commit message: updateboard, added seekcurrenttest
Parts:
- removed C2: 10nF, Capacitor_SMD:C_0402_1005Metric, symbol ALPACARepeaterLibrary:10nF
- removed D1: D_Schottky, primecamLNABiasPotVreg:DO-214BA_MCH, symbol Device:D_Schottky
- removed R10: 2150, Resistor_SMD:R_0603_1608Metric, symbol ALPACA:10k
- removed R11, R12, R15, R16: 10K, Resistor_SMD:R_0603_1608Metric, symbol ALPACA:10k
- removed R13, R14: 5.1K, Resistor_SMD:R_0603_1608Metric, symbol ALPACA:5.1k
- removed R9: 1370, Resistor_SMD:R_0603_1608Metric, symbol ALPACA:10k
- removed U2: LTC4302-1, Package_SO:MSOP-10_3x3mm_P0.5mm, symbol ALPACA:LTC4302-1
- added R166: 0, Resistor_SMD:R_0402_1005Metric, symbol Device:R
- added R41: 1k, Resistor_SMD:R_0603_1608Metric, symbol Device:R
- added R49: 43, Resistor_SMD:R_1206_3216Metric, symbol Device:R
- added U2: CPC1002NTR, Package_SO:SOP-4_3.8x4.1mm_P2.54mm, symbol LNA_Bias:CPC1002NTR
- C11, C8: LCSC Part # KAM05ACG1H100JH -> C32949; Part (none) -> CL05C100JB5NNNC
- C12: LCSC Part # TR3B106K025C0450 -> C1952910; Part (none) -> T494B106M016AT
- C13, C14, C4, C6: LCSC Part # EMF105B7104KVHF -> C1525; Part (none) -> CL05B104KO5NNNC
- C3, C9: LCSC Part # 0603YD106MAT2A -> C19702; Part (none) -> CL10A106KP8NNNC
- C5: LCSC Part # C0402C475K8PACTU -> C23733; Part (none) -> CL05A475MP5NRNC
- R17: LCSC Part # SDR03EZPD1202 -> C8218; Part (none) -> 0603WAF2000T5E
- R18: value 3k65 -> 1k; LCSC Part # CPF0603F3K65C1 -> C21190; Part (none) -> 0603WAF1001T5E
- R19: LCSC Part # (none) -> C21190; Part (none) -> 0603WAF1001T5E
- R20, R22: LCSC Part # TNPW060310R0BETA -> C22859; Part (none) -> 0603WAF100JT5E
- R21: value 10 -> DNI; now not fitted
- R23: LCSC Part # RT1206BRD071RL -> C1857715; Link https://www.mouser.com/ProductDetail/YAGEO/RT1206BRD071RL?q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 -> https://jlcpcb.com/parts/componentSearch?searchTxt=TNPW1206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; Part (none) -> TNPW12061R00DEEA
- RV1: now not fitted
- TP1: LCSC Part # 5006 -> C5199811; Part (none) -> RH-5006
- TP2: LCSC Part # 5006 -> C2906763; Mouser 534-5006 -> 534-5005; Part (none) -> 5005
- U3: LCSC Part # AD5144BCPZ100-RL7 -> C577979; Part (none) -> AD5144BCPZ100-RL7
- U4: LCSC Part # LT3080EDD-1#TRPBF -> C462675; Part (none) -> LT3080EDD#TRPBF
- U5: value AQY212G3HS -> CPC1002NTR; LCSC Part # AQY212G3HS -> C5359028; Link https://www.mouser.com/ProductDetail/Panasonic-Industrial-D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 -> https://www.digikey.com/en/products/detail/littelfuse-inc/C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; Mouser 769-AQY212G3HS -> 849-CPC1002NTR; Part (none) -> CPC1002NTR
- U6: LCSC Part # INA219BIDR -> C138706; Part (none) -> INA219AIDR
Connections:
- net 5V: now also R41.1; no longer R18.2
- net BIAS_OUT_CH${ChanNum}: now also U2.4
- net GND: now also R49.2; no longer U3.21 (ADDR1), U3.22 (ADDR0), U6.1 (A1), U6.2 (A0)
- net at C5.1, RV1.1, U4.4 (SET): now also R166.1
- net at R21.2, RV1.2, RV1.3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: now also R166.2
- net at U5.3: now also R19.1, R20.2, R23.1
- net GPIO1 renamed Ch${ChanNum}_En
- net SCL${ChanNum} renamed SCL
- net SDA${ChanNum} renamed SDA
- new net: R41.2, U2.1
- new net: R49.1, U2.3
- new net ${INA-A0}: U6.2 (A0)
- new net ${INA-A1}: U6.1 (A1)
- new net ${POT-A0}: U3.22 (ADDR0)
- new net ${POT-A1}: U3.21 (ADDR1)
- new net Ch${ChanNum}_TestLoad_En: U2.2
- new net LED${ChanNum}: R18.2
Other:
- note added: "Channel: ${ChanNum}"
