File: board/primecamLNABiasPotVreg.kicad_sch (KiCad schematic)
At the start: 14 parts, among them J3 Conn_01x03, U1 LTC4302-1

Commit message: updateboard, added seekcurrenttest
Parts:
- removed J3: Conn_01x03, Connector_PinHeader_2.54mm:PinHeader_1x03_P2.54mm_Vertical, symbol Connector_Generic:Conn_01x03
- added BAR1: H204CGDL, primecamLNABiasPotVreg:H204CGDL, symbol LNA_Bias:H204CGDL
- added C15: 0.1u, Capacitor_SMD:C_0402_1005Metric, symbol ASTHROS_IF_OUTPUT_AMP-rescue:0.1u-ASTHROS_IF_OUTPUT_AMP
- added C24, C25: 10u, Capacitor_SMD:C_0603_1608Metric, symbol ALPACA:10u
- added D1: LED, ALPACA:LED_Dialight_551, symbol Device:LED
- added J4: VME_CARD_03X32, ALPACA:DIN41612_B_3x32_Horizontal, symbol ALPACA:VME_CARD_03X32
- added J5: DB25_Pins_MountingHoles, primecamLNABiasPotVreg:TE_5747842-4, symbol Connector:DB25_Pins_MountingHoles
- added R10, R11, R12, R13, R14, R15, R16, R24, R25, R26, R27, R28, R29, R30, R31, R39, R9: 10K, Resistor_SMD:R_0603_1608Metric, symbol ALPACA:10k
- added TP10, TP11, TP24, TP25, TP8, TP9: TestPoint, TestPoint:TestPoint_Keystone_5005-5009_Compact, symbol Connector:TestPoint
- added U12: PCF8575, Package_SO:SSOP-24_5.3x8.2mm_P0.65mm, symbol LNA_Bias:PCF8575
- C1: LCSC Part # 04025Z103KAT2A -> C15195; Part (none) -> CL05B103KB5NNNC
- R1: Part (none) -> RA73F1J2K8BTDF
- R2: Part (none) -> ERA-3VEB1370V
- R3, R4, R7: LCSC Part # RNCF0603TKY10K0 -> C15401; Part (none) -> 0603WAJ0103T5E; Part Number (none) -> 10K
- R5, R6: LCSC Part # ERJ-3EKF5101V -> C23186; Part (none) -> 0603WAF5101T5E
- R8: value 10K -> 1k6; LCSC Part # RNCF0603TKY10K0 -> C22847; Part (none) -> 0603WAF1601T5E
- TP4: LCSC Part # 5006 -> C5277088; Mouser 534-5006 -> 534-5009; Part (none) -> RH-5009
- TP5, TP6: LCSC Part # 5006 -> C5277087; Mouser 534-5006 -> 534-5008; Part (none) -> RH-5008
- U1: LCSC Part # LTC4302CMS-1#PBF -> C688009; Part (none) -> LTC4302CMS-1#TRPBF
Connections:
- net 12V: now also C25.1, J4.C31 (+12v), TP11.1; no longer TP5.1
- net 5V: now also BAR1.10 (A), BAR1.12 (A), BAR1.14 (A), BAR1.16 (A), BAR1.2 (A), BAR1.4 (A), BAR1.6 (A), BAR1.8 (A), C15.1, C24.1, J4.A32 (+5v), J4.B32 (+5v), J4.C32 (+5v), R10.2, R11.2, R12.2, R13.2, R14.2, R15.2, R16.2, R24.1, R25.2, R26.2, R27.2, R28.2, R29.2, R30.2, R31.2, R39.2, R9.2, TP25.1, U12.2 (A1), U12.21 (A0), U12.24 (VCC), U12.3 (A2); no longer TP4.1
- net BIAS_OUT_CH1: now also J5.9
- net BIAS_OUT_CH2: now also J5.8
- net GND: now also C15.2, C24.2, C25.2, J4.A11 (GND), J4.A15 (GND), J4.A17 (GND), J4.A19 (GND), J4.A9 (GND), J4.B20 (GND), J4.B23 (GND), J4.C9 (GND), J5.0 (PAD), J5.1, J5.13, J5.14 (P14), J5.15 (P15), J5.16 (P16), J5.17 (P17), J5.18 (P18), J5.19 (P19), J5.20 (P20), J5.21 (P21), J5.22 (P22), J5.23 (P23), J5.24 (P24), J5.25 (P25), TP10.1, TP24.1, U12.12 (GND); no longer TP6.1
- net SCL_LTC0: now also J4.B21 (SERCLK), TP8.1
- net SDA_LTC0: now also TP6.1, J4.B22 (SERDAT*)
- net boardAddr: now reaches R1.2, R2.1, U1.4 (ADD)
- net boardAddr: now also J4.B4 (BG0IN*), TP9.1
- net at U1.6 (GPIO1): now also D1.1; no longer R8.2
- net SCL_BiasCircuit renamed SCL
- net SCL: now also TP4.1, U12.22 (SCL)
- net SDA_BiasCircuit renamed SDA
- net SDA: now also TP5.1, U12.23 (SDA)
- new net: D1.2, R8.2
- new net: R24.2, U12.1 (~{INT})
- new net -12V: J4.A31 (-12v)
- new net BIAS_OUT_CH3: J5.7
- new net BIAS_OUT_CH4: J5.6
- new net BIAS_OUT_CH5: J5.5
- new net BIAS_OUT_CH6: J5.4
- new net BIAS_OUT_CH7: J5.3
- new net BIAS_OUT_CH8: J5.2
- new net Ch1_En: R16.1, U12.4 (P0)
- new net Ch1_TestLoad_En: R25.1, U12.13 (P10)
- new net Ch2_En: R15.1, U12.5 (P1)
- new net Ch2_TestLoad_En: R26.1, U12.14 (P11)
- new net Ch3_En: R14.1, U12.6 (P2)
- new net Ch3_TestLoad_En: R27.1, U12.15 (P12)
- new net Ch4_En: R13.1, U12.7 (P3)
- new net Ch4_TestLoad_En: R28.1, U12.16 (P13)
- new net Ch5_En: R12.1, U12.8 (P4)
- new net Ch5_TestLoad_En: R29.1, U12.17 (P14)
- new net Ch6_En: R11.1, U12.9 (P5)
- new net Ch6_TestLoad_En: R30.1, U12.18 (P15)
- new net Ch7_En: R10.1, U12.10 (P6)
- new net Ch7_TestLoad_En: R31.1, U12.19 (P16)
- new net Ch8_En: R9.1, U12.11 (P7)
- new net Ch8_TestLoad_En: R39.1, U12.20 (P17)
- new net LED1: BAR1.1 (K)
- new net LED2: BAR1.3 (K)
- new net LED3: BAR1.5 (K)
- new net LED4: BAR1.7 (K)
- new net LED5: BAR1.9 (K)
- new net LED6: BAR1.11 (K)
- new net LED7: BAR1.13 (K)
- new net LED8: BAR1.15 (K)
Other:
- removed sheet BiasCircuit
- added sheet BiasCircuit2 (BiasCircuit.kicad_sch)
- added sheet BiasCircuit3 (BiasCircuit.kicad_sch)
- added sheet BiasCircuit4 (BiasCircuit.kicad_sch)
- added sheet BiasCircuit5 (BiasCircuit.kicad_sch)
- added sheet BiasCircuit6 (BiasCircuit.kicad_sch)
- added sheet BiasCircuit7 (BiasCircuit.kicad_sch)
- added sheet BiasCircuit8 (BiasCircuit.kicad_sch)
- sheet BiasCircuit1 ports: added LED${ChanNum}; removed SCL_BiasCircuit, SDA_BiasCircuit
- note added: "Per-Card Address Table"
- note added: "WARNING: TEST LOAD RESISTOR HAS INCORRECT JLC PART NUMBER -SHOULD BE 43 OHM, IS 0.001 OHM"
- note removed: "BACKPLANE CARD 1 OF 18"
- note removed: "BACKPLANE CARD n OF 18"
- note removed: "Raspberry PI & Daughterboard"
- note removed: "SDA_LTC... SCL_LTC..."
- note removed: "SDA_LTC0 SCL_LTC0"
- note removed: "SDA_LTC1 SCL_LTC1"
- note removed: "SDA_LTC19 SCL_LTC19"
- note removed: "SDA_LTC31 SCL_LTC31"
- note removed: "SDA_LTCn SCL_LTCn"
- note removed: "SDA_PI SCL_PI"
- note removed: "SERCOM"
- company: (none) -> Arizona State University
- moved on the sheet: C1, R1, R2, R3, R4, R5, R6, R7, R8, U1
